File: USB_power.kicad_sch (KiCad schematic)
At the start: 33 parts, among them J1 PWR_IN, J2 USB_A_Stacked, J3 Power_check, J4 USB_C_Receptacle_USB2.0_16P, J5 USB_A_Stacked, SW1 Switch

Commit message: 穴のシンボル変更
Parts:
- F1: value Fuse -> 10A
- H1, H2, H3, H4: symbol Mechanical:MountingHole -> Mechanical:MountingHole_Pad
Connections:
- no-connect marks 29 -> 33
Changed lines of the file:
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@@
 	)
 	(no_connect
+		(at 135.89 168.91)
+	)
+	(no_connect
 		(at 219.71 66.04)
 	)
@@
 	)
 	(no_connect
+		(at 78.74 168.91)
+	)
+	(no_connect
 		(at 74.93 74.93)
 	)
@@
 	)
 	(no_connect
+		(at 97.79 168.91)
+	)
+	(no_connect
+		(at 116.84 168.91)
+	)
+	(no_connect
 		(at 219.71 83.82)
 	)
@@
 	)
 	(symbol
-		(lib_id "Mechanical:MountingHole")
-		(at 247.65 125.73 0)
+		(lib_id "Mechanical:MountingHole_Pad")
+		(at 116.84 166.37 0)
 		(unit 1)
 		(exclude_from_sim yes)
@@
 		(fields_autoplaced yes)
 		(property "Reference" "H3"
-			(at 250.19 124.4599 0)
+			(at 119.38 163.8299 0)
 			(effects
 				(font
@@
 		)
 		(property "Value" "MountingHole"
-			(at 250.19 126.9999 0)
+			(at 119.38 166.3699 0)
 			(effects
 				(font
@@
 		)
 		(property "Footprint" "MountingHole:MountingHole_3.2mm_M3_Pad_Via"
-			(at 247.65 125.73 0)
+			(at 116.84 166.37 0)
 			(effects
 				(font
@@
 		)
 		(property "Datasheet" "~"
-			(at 247.65 125.73 0)
+			(at 116.84 166.37 0)
 			(effects
 				(font
@@
 			)
 		)
-		(property "Description" "Mounting Hole without connection"
-			(at 247.65 125.73 0)
+		(property "Description" "Mounting Hole with connection"
+			(at 116.84 166.37 0)
 			(effects
 				(font
@@
 			)
 		)
+		(pin "1"
+		)
 		(instances
 			(project ""
@@
 			)
 		)
-		(property "Value" "Fuse"
+		(property "Value" "10A"
 			(at 46.99 78.7399 0)
 			(effects
@@
 	)
 	(symbol
-		(lib_id "Mechanical:MountingHole")
-		(at 247.65 133.35 0)
+		(lib_id "Mechanical:MountingHole_Pad")
+		(at 135.89 166.37 0)
 		(unit 1)
 		(exclude_from_sim yes)
@@
 		(fields_autoplaced yes)
 		(property "Reference" "H4"
-			(at 250.19 132.0799 0)
+			(at 138.43 163.8299 0)
 			(effects
 				(font
@@
 		)
 		(property "Value" "MountingHole"
-			(at 250.19 134.6199 0)
+			(at 138.43 166.3699 0)
 			(effects
 				(font
@@
 		)
 		(property "Footprint" "MountingHole:MountingHole_3.2mm_M3_Pad_Via"
-			(at 247.65 133.35 0)
+			(at 135.89 166.37 0)
 			(effects
 				(font
@@
 		)
 		(property "Datasheet" "~"
-			(at 247.65 133.35 0)
+			(at 135.89 166.37 0)
 			(effects
 				(font
@@
 			)
 		)
-		(property "Description" "Mounting Hole without connection"
-			(at 247.65 133.35 0)
+		(property "Description" "Mounting Hole with connection"
+			(at 135.89 166.37 0)
 			(effects
 				(font
@@
 			)
 		)
+		(pin "1"
+		)
 		(instances
 			(project ""
@@
 	)
 	(symbol
-		(lib_id "Mechanical:MountingHole")
-		(at 247.65 118.11 0)
+		(lib_id "Mechanical:MountingHole_Pad")
+		(at 97.79 166.37 0)
 		(unit 1)
 		(exclude_from_sim yes)
@@
 		(fields_autoplaced yes)
 		(property "Reference" "H2"
-			(at 250.19 116.8399 0)
+			(at 100.33 163.8299 0)
 			(effects
 				(font
@@
 		)
 		(property "Value" "MountingHole"
-			(at 250.19 119.3799 0)
+			(at 100.33 166.3699 0)
 			(effects
 				(font
@@
 		)
 		(property "Footprint" "MountingHole:MountingHole_3.2mm_M3_Pad_Via"
-			(at 247.65 118.11 0)
+			(at 97.79 166.37 0)
 			(effects
 				(font
@@
 		)
 		(property "Datasheet" "~"
-			(at 247.65 118.11 0)
+			(at 97.79 166.37 0)
 			(effects
 				(font
@@
 			)
 		)
-		(property "Description" "Mounting Hole without connection"
-			(at 247.65 118.11 0)
+		(property "Description" "Mounting Hole with connection"
+			(at 97.79 166.37 0)
 			(effects
 				(font
@@
 			)
 		)
+		(pin "1"
+		)
 		(instances
 			(project ""
@@
 	)
 	(symbol
-		(lib_id "Mechanical:MountingHole")
-		(at 247.65 110.49 0)
+		(lib_id "Mechanical:MountingHole_Pad")
+		(at 78.74 166.37 0)
 		(unit 1)
 		(exclude_from_sim yes)
@@
 		(on_board yes)
 		(dnp no)
-		(fields_autoplaced yes)
 		(property "Reference" "H1"
-			(at 250.19 109.2199 0)
+			(at 81.28 163.8299 0)
 			(effects
 				(font
@@
 		)
 		(property "Value" "MountingHole"
-			(at 250.19 111.7599 0)
+			(at 81.28 166.3699 0)
 			(effects
 				(font
@@
 		)
 		(property "Footprint" "MountingHole:MountingHole_3.2mm_M3_Pad_Via"
-			(at 247.65 110.49 0)
+			(at 78.74 166.37 0)
 			(effects
 				(font
@@
 		)
 		(property "Datasheet" "~"
-			(at 247.65 110.49 0)
+			(at 78.74 166.37 0)
 			(effects
 				(font
@@
 			)
 		)
-		(property "Description" "Mounting Hole without connection"
-			(at 247.65 110.49 0)
+		(property "Description" "Mounting Hole with connection"
+			(at 78.74 166.37 0)
 			(effects
 				(font
@@
 			)
 		)
+		(pin "1"
+		)
 		(instances
